Commit message: feat:Add structure in rviz2

File: src/articubot_one/description/gazebo_control.xacro (robot description, xacro)
@@ -2,39 +2,54 @@
 <robot xmlns:xacro="http://www.ros.org/wiki/xacro">
 <gazebo>
-    <plugin name="diff_drive" filename="libgazebo_ros_diff_drive.so">
-        <!-- Wheel Information - Front wheels driven -->
-        <left_joint>front_left_wheel_joint</left_joint>
-        <right_joint>front_right_wheel_joint</right_joint>
-        <wheel_separation>0.35</wheel_separation>
-        <wheel_diameter>0.1</wheel_diameter>
-        <!-- Limits -->
-        <max_wheel_torque>200</max_wheel_torque>
-        <max_wheel_acceleration>10.0</max_wheel_acceleration>
-        <!-- Topic names (ROS2) -->
-        <command_topic>cmd_vel</command_topic>
-        <odometry_topic>odom</odometry_topic>
-        <!-- Output -->
-        <odometry_frame>odom</odometry_frame>
-        <robot_base_frame>base_link</robot_base_frame>
-        <publish_odom>true</publish_odom>
-        <publish_odom_tf>true</publish_odom_tf>
-        <publish_wheel_tf>true</publish_wheel_tf>
-        <!-- ROS2 specific -->
-        <ros>
-            <namespace>/</namespace>
-            <remapping>cmd_vel:=cmd_vel</remapping>
-            <remapping>odom:=odom</remapping>
-        </ros>
-    </plugin>
+<plugin name="diff_drive" filename="libgazebo_ros_diff_drive.so">
+    <!-- Wheel Information - Front wheels driven -->
+    <left_joint>front_left_wheel_joint</left_joint>
+    <right_joint>front_right_wheel_joint</right_joint>
+    <wheel_separation>0.35</wheel_separation>
+    <wheel_diameter>0.1</wheel_diameter>
+    <!-- Limits -->
+    <max_wheel_torque>200</max_wheel_torque>
+    <max_wheel_acceleration>10.0</max_wheel_acceleration>
+    <!-- Topic names (ROS2) -->
+    <command_topic>cmd_vel</command_topic>
+    <odometry_topic>odom</odometry_topic>
+    <!-- Output -->
+    <odometry_frame>odom</odometry_frame>
+    <robot_base_frame>base_link</robot_base_frame>
+    <publish_odom>true</publish_odom>
+    <publish_odom_tf>true</publish_odom_tf>
+    <publish_wheel_tf>true</publish_wheel_tf>
+    <!-- ROS2 specific -->
+    <ros>
+        <namespace>/</namespace>
+        <remapping>cmd_vel:=cmd_vel</remapping>
+        <remapping>odom:=odom</remapping>
+    </ros>
+</plugin>
+</gazebo>
+<!-- ADD THESE: Front wheels need good friction for driving -->
+<gazebo reference="front_left_wheel">
+    <mu1>1.0</mu1>
+    <mu2>1.0</mu2>
+    <kp>1000000.0</kp>
+    <kd>100.0</kd>
+    <material>Gazebo/Blue</material>
+</gazebo>
+<gazebo reference="front_right_wheel">
+    <mu1>1.0</mu1>
+    <mu2>1.0</mu2>
+    <kp>1000000.0</kp>
+    <kd>100.0</kd>
+    <material>Gazebo/Blue</material>
 </gazebo>
 <!-- Make rear wheels have low friction so they roll freely -->
 <gazebo reference="rear_left_wheel">
-    <mu1 value="0.1"/>
-    <mu2 value="0.1"/>
+    <mu1>0.1</mu1>
+    <mu2>0.1</mu2>
     <material>Gazebo/Blue</material>
 </gazebo>
 <gazebo reference="rear_right_wheel">
-    <mu1 value="0.1"/>
-    <mu2 value="0.1"/>
+    <mu1>0.1</mu1>
+    <mu2>0.1</mu2>
     <material>Gazebo/Blue</material>
 </gazebo>

File: src/articubot_one/description/robot.urdf.xacro (robot description, xacro)
@@ -3,3 +3,5 @@
     <xacro:include filename="robot_core.xacro" />
     <xacro:include filename="gazebo_control.xacro" />
+    <xacro:include filename="lidar.xacro" />
+    <xacro:include filename="inertial_macros.xacro" />
 </robot>

Commit message: feat:Complete mapping feature

File: src/articubot_one/description/gazebo_control.xacro (robot description, xacro)
@@ -3,54 +3,64 @@
 <gazebo>
 <plugin name="diff_drive" filename="libgazebo_ros_diff_drive.so">
-    <!-- Wheel Information - Front wheels driven -->
-    <left_joint>front_left_wheel_joint</left_joint>
-    <right_joint>front_right_wheel_joint</right_joint>
-    <wheel_separation>0.35</wheel_separation>
-    <wheel_diameter>0.1</wheel_diameter>
-    <!-- Limits -->
-    <max_wheel_torque>200</max_wheel_torque>
-    <max_wheel_acceleration>10.0</max_wheel_acceleration>
-    <!-- Topic names (ROS2) -->
-    <command_topic>cmd_vel</command_topic>
-    <odometry_topic>odom</odometry_topic>
-    <!-- Output -->
-    <odometry_frame>odom</odometry_frame>
-    <robot_base_frame>base_link</robot_base_frame>
-    <publish_odom>true</publish_odom>
-    <publish_odom_tf>true</publish_odom_tf>
-    <publish_wheel_tf>true</publish_wheel_tf>
-    <!-- ROS2 specific -->
-    <ros>
-        <namespace>/</namespace>
-        <remapping>cmd_vel:=cmd_vel</remapping>
-        <remapping>odom:=odom</remapping>
-    </ros>
+<!-- Wheel Information - Front wheels driven -->
+<update_rate>50</update_rate>
+<left_joint>front_left_wheel_joint</left_joint>
+<right_joint>front_right_wheel_joint</right_joint>
+<wheel_separation>0.35</wheel_separation>
+<wheel_diameter>0.1</wheel_diameter>
+<!-- Limits -->
+<max_wheel_torque>200</max_wheel_torque>
+<max_wheel_acceleration>10.0</max_wheel_acceleration>
+<!-- Topic names (ROS2) -->
+<command_topic>cmd_vel</command_topic>
+<!-- Output -->
+<publish_odom>true</publish_odom>
+<publish_odom_tf>true</publish_odom_tf>
+<publish_wheel_tf>true</publish_wheel_tf>
+<odometry_frame>odom</odometry_frame>
+<robot_base_frame>base_link</robot_base_frame>
+<!-- ROS2 specific -->
+<ros>
+<namespace>/</namespace>
+<remapping>cmd_vel:=cmd_vel</remapping>
+<remapping>odom:=odom</remapping>
+</ros>
 </plugin>
 </gazebo>
-<!-- ADD THESE: Front wheels need good friction for driving -->
+<!-- Front wheels need good friction for driving -->
 <gazebo reference="front_left_wheel">
-    <mu1>1.0</mu1>
-    <mu2>1.0</mu2>
-    <kp>1000000.0</kp>
-    <kd>100.0</kd>
-    <material>Gazebo/Blue</material>
+<mu1>1.0</mu1>
+<mu2>1.0</mu2>
+<kp>1000000.0</kp>
+<kd>100.0</kd>
+<minDepth>0.001</minDepth>
+<maxVel>0.1</maxVel>
+<material>Gazebo/Blue</material>
 </gazebo>
 <gazebo reference="front_right_wheel">
-    <mu1>1.0</mu1>
-    <mu2>1.0</mu2>
-    <kp>1000000.0</kp>
-    <kd>100.0</kd>
-    <material>Gazebo/Blue</material>
+<mu1>1.0</mu1>
+<mu2>1.0</mu2>
+<kp>1000000.0</kp>
+<kd>100.0</kd>
+<minDepth>0.001</minDepth>
+<maxVel>0.1</maxVel>
+<material>Gazebo/Blue</material>
 </gazebo>
 <!-- Make rear wheels have low friction so they roll freely -->
 <gazebo reference="rear_left_wheel">
-    <mu1>0.1</mu1>
-    <mu2>0.1</mu2>
-    <material>Gazebo/Blue</material>
+<mu1>0.1</mu1>
+<mu2>0.1</mu2>
+<kp>1000000.0</kp>
+<kd>10.0</kd>
+<minDepth>0.001</minDepth>
+<material>Gazebo/Blue</material>
 </gazebo>
 <gazebo reference="rear_right_wheel">
-    <mu1>0.1</mu1>
-    <mu2>0.1</mu2>
-    <material>Gazebo/Blue</material>
+<mu1>0.1</mu1>
+<mu2>0.1</mu2>
+<kp>1000000.0</kp>
+<kd>10.0</kd>
+<minDepth>0.001</minDepth>
+<material>Gazebo/Blue</material>
 </gazebo>
 </robot>
