Commit message: feat:Add GPIO connection

File: src/articubot_one/description/robot_core.xacro (robot description, xacro)
@@ -4,4 +4,12 @@
 <link name="base_link">
 </link>
+  <!-- BASE_FOOTPRINT LINK -->
+    <joint name="base_footprint_joint" type="fixed">
+        <parent link="base_link"/>
+        <child link="base_footprint"/>
+        <origin xyz="0 0 0" rpy="0 0 0"/>
+    </joint>
+    <link name="base_footprint">
+    </link>
 <!-- CHASSIS LINK -->
 <joint name="chassis_joint" type="fixed">
